File: fyp-esc.kicad_sch (KiCad schematic)
At the start: 53 parts, among them U1 STM32F405RGT6

Commit message: Schematic organisation
Parts:
- added C? (x3): C_Small, symbol Device:C_Small
- added C? (x2): 10u, symbol Device:C_Small
- added R?: 1k, symbol Device:R_Small
Connections:
- net VDRAIN is gone; now on net +BATT: C?.1, U?.6 (VDRAIN)
- net +3.3VA: now also R?.2
- net +BATT: now also C?.2, C?.2
- net DRV:SDO: now also R?.1
- net GND: now also C?.1, C?.1
- net nFAULT renamed DRV:nFAULT
Other:
- note added: "Bulk"
- note added: "Bypass"
- note added: "CANBUS"
- note added: "Connectors"
- note added: "I2C"
- note added: "UART"
- note added: "USB"
- moved on the sheet: C?, Cb, Cbyp, Cff, Cin, Cinx, Cout, D1, D?, F?, FB?, L1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

Commit message: stm32 pinout & connectors
Parts:
- added D?: RedLED, symbol Device:LED_Small
- added H? (x4): MountingHole_Pad, symbol Mechanical:MountingHole_Pad
- added J?: UART, symbol Connector_Generic:Conn_01x04
- added J?: USB_C_Receptacle_USB2.0, Connector_USB:USB_C_Receptacle_HRO_TYPE-C-31-M-12, symbol Connector:USB_C_Receptacle_USB2.0
- added J?: SWD, symbol Connector_Generic:Conn_02x05_Odd_Even
- added J?: I2C, symbol Connector_Generic:Conn_01x04
- added R? (x2): 5k1, symbol Device:R_Small
- added R?: 1k, symbol Device:R_Small
- added R? (x2): 4k7, symbol Device:R_Small
- added U?: USBLC6-2SC6, Package_TO_SOT_SMD:SOT-23-6, symbol Power_Protection:USBLC6-2SC6
Connections:
- net DGND is gone; now on net GND: C?.2, U?.41 (DGND)
- net SHA is gone; now on net MOTA: U?.9 (SHA)
- net SHB is gone; now on net MOTB: U?.16 (SHB)
- net SHC is gone; now on net MOTC: U?.19 (SHC)
- net SNA is gone; now on net GND: U?.12 (SNA)
- net SNB is gone; now on net GND: U?.13 (SNB)
- net SNC is gone; now on net GND: U?.22 (SNC)
- net +3.3VA: now also D?.2 (A), J?.1 (Pin_1), J?.1 (Pin_1), J?.1 (Pin_1), R?.1, R?.1
- net +BATT: now also C?.2, C?.2, C?.2, Q?.2 (D), Q?.2 (D), Q?.2 (D)
- net DRV:SCLK: now also U1.21 (PA5)
- net DRV:SDI: now also U1.23 (PA7)
- net DRV:SDO: now also U1.22 (PA6)
- net DRV:nSCS: now also U1.24 (PC4)
- net GHA: now also Q?.1 (G)
- net GHB: now also Q?.1 (G)
- net GHC: now also Q?.1 (G)
- net GLB: now also Q?.1 (G)
- net GLC: now also Q?.1 (G)
- net GND: now also C?.1, C?.1, C?.1, R?.2, R?.2, R?.2, H?.1, H?.1, H?.1, H?.1, J?.3 (Pin_3), J?.4 (Pin_4), J?.4 (Pin_4), J?.5 (Pin_5), J?.9 (Pin_9), J?.A1 (GND), J?.A12 (GND), J?.B1 (GND), J?.B12 (GND), J?.S1 (SHIELD), R?.2, R?.2, R?.2, U?.2 (GND)
- net MOTA: now also Q?.2 (D), Q?.3 (S)
- net MOTB: now also Q?.2 (D), Q?.3 (S)
- net MOTC: now also Q?.2 (D), Q?.3 (S)
- net SPA: now also Q?.3 (S), R?.1
- net SPB: now also Q?.3 (S), R?.1
- net SPC: now also Q?.3 (S), R?.1
- net USB_D+: now also U1.45 (PA12), U?.4 (I/O2)
- net USB_D-: now also U1.44 (PA11), U?.6 (I/O1)
- net ENC_CH1: now reaches U1.14 (PA0)
- net ENC_CH2: now reaches U1.15 (PA1)
- net SWDIO: now reaches U1.46 (PA13)
- net SWDIO: now also J?.2 (Pin_2)
- net SWCLK: now reaches U1.49 (PA14)
- net SWCLK: now also J?.4 (Pin_4)
- net USART3_TX: now reaches U1.51 (PC10)
- net USART3_TX: now also J?.2 (Pin_2)
- net USART3_RX: now reaches U1.52 (PC11)
- net USART3_RX: now also J?.3 (Pin_3)
- net SWO: now reaches U1.55 (PB3)
- net SWO: now also J?.6 (Pin_6)
- net CAN1_RX: now reaches U1.61 (PB8)
- net CAN1_TX: now reaches U1.62 (PB9)
- net ENABLE renamed DRV:ENABLE
- net NRST renamed nRST
- net nRST: now also J?.10 (Pin_10)
- new net: J?.A7 (D-), J?.B7 (D-), U?.1 (I/O1)
- new net: J?.A6 (D+), J?.B6 (D+), U?.3 (I/O2)
- new net: J?.A5 (CC1), R?.1
- new net: J?.B5 (CC2), R?.1
- new net: D?.1 (K), R?.1
- new net I2C1_SCL: J?.2 (Pin_2), R?.2
- new net I2C1_SDA: J?.3 (Pin_3), R?.2
- new net USB_Vbus: J?.A4 (VBUS), J?.A9 (VBUS), J?.B4 (VBUS), J?.B9 (VBUS), U?.5 (VBUS)
- no-connect marks 0 -> 4
Other:
- note added: "3V drop over LED 3.3V - 3V = 0.3V 1kOhm -> 0.3/1k = 0.3mA"
- note added: "5.1k resistors denote this as a "downstream" USB C port, i.e. device not host"
- note added: "Battery Input 12 - 75V"
- note added: "CAN"
- note added: "Datasheet p66"
- note added: "EN from MCU"
- note added: "ENCODER"
- note added: "ESD protection"
- note added: "FAULT to MCU"
- note added: "Gate control from MCU"
- note added: "Gate outputs to MOSFETs"
- note added: "LM5008A"
- note added: "Power LED: 2V drop over LED 3.3V - 2V = 1.3V 4.7kOhm -> 1.3/4.7k = 0.277mA"
- note added: "SOx feedback to MCU"
- note added: "SPI to MCU"
- note added: "SWD"
- note added: "Thermal Pad"
- note added: "USB Input 5V"
- note removed: "3V drop over LED 3.3V - 3V = 0.3V 3kOhm -> 0.3/1k = 0.3mA"
- note removed: "CANBUS"
- note removed: "Input 12 - 75V"
- moved on the sheet: C?, D?, F?, FB?, R?, Y?

Commit message: ESC schematic v1 symbol placement finished
dual USB/BATT MCU PSU,
CAN connector,
Encoder connector.
Parts:
- added C?: 0.1u, symbol Device:C_Small
- added C?: 47n, symbol Device:C_Small
- added D? (x2): D_Z, symbol Device:D_Zener_Small
- added IC?: MAX33041EASA+, SOIC127P600X175-8N, symbol SamacSys_Parts:MAX33041EASA+
- added J?: ENC, symbol Connector_Generic:Conn_01x04
- added J?: CAN, symbol Connector_Generic:Conn_01x04
- added Q? (x2): Q_PMOS_GDS, symbol Device:Q_PMOS_GDS
- added R? (x2): 100k, symbol Device:R_Small
- added R? (x2): 60, symbol Device:R_Small
- added U?: AMS1117-3.3, Package_TO_SOT_SMD:SOT-223-3_TabPin2, symbol Regulator_Linear:AMS1117-3.3
- FB?: value 600ohm @ 100MHz -> 600ohm@100MHz
- R?: value 1k -> 4K7
Connections:
- net CAN1_RX is gone; now on net I2C1_SCL: U1.61 (PB8)
- net CAN1_TX is gone; now on net I2C1_SDA: U1.62 (PB9)
- net +3.3VA: now also C?.1, IC?.3 (VDD), J?.1 (Pin_1), J?.1 (Pin_1), U?.2 (VO)
- net +BATT: now also D?.2 (A), Q?.1 (G), R?.1
- net ENC_CH1: now also J?.2 (Pin_2)
- net ENC_CH2: now also J?.3 (Pin_3)
- net GND: now also C?.2, C?.2, IC?.2 (GND), IC?.8 (STBY), J?.4 (Pin_4), J?.4 (Pin_4), R?.2, R?.2, U?.1 (GND)
- net USB_Vbus: now also Q?.2 (D)
- net VIN: now also FB?.2
- net CAN2_RX: now reaches U1.57 (PB5)
- net CAN2_RX: now also IC?.4 (RXD)
- net CAN2_TX: now reaches U1.58 (PB6)
- net CAN2_TX: now also IC?.1 (TXD)
- net CAN:SHDN: now reaches U1.59 (PB7)
- net CAN:SHDN: now also IC?.5 (SHDN)
- net at FB?.1: now also D?.1 (K), Q?.3 (S)
- net at F?.1: now also Q?.2 (D)
- new net: D?.2 (A), Q?.1 (G), R?.1
- new net: C?.1, R?.1, R?.2
- new net: D?.1 (K), Q?.3 (S), U?.3 (VI)
- new net: IC?.6 (CANL), J?.3 (Pin_3), R?.2
- new net: IC?.7 (CANH), J?.2 (Pin_2), R?.1
Other:
- note added: "3.3V LDO"
- note added: "<- ESD protection"
- note added: "Datasheet p16: STBY high -> standby ∴ STBY -> GND"
- note added: "If+BATT voltage is present, then: PMOS reverse biased and turns off ∴ draw from USB 5V disabled so no PSU backfeeding occurs (and damages USB)"
- note added: "Initial HF filtering"
- note added: "Vout taken between RC to reduce output voltage ripple at the expense of degraded load regulation (okay since MCU load is fairly constant)"
- note added: "Zener diode limits Vgs to within datasheet limit"
- note removed: "ESD protection"
- note removed: "Initial filtering"
- note removed: "Vout taken between RC to reduce output voltage ripple at the expense of degraded load regulation (fine since MCU load is fairly constant)"
- moved on the sheet: Cb, Cbyp, Cff, Cin, Cinx, Cout, D1, D?, F?, FB?, H?, J?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

Commit message: BOM / component selection
Parts:
- removed D1: 900m, symbol Device:D_Small
- removed Q? (x2): Q_PMOS_GDS, symbol Device:Q_PMOS_GDS
- added D1: 900m, Diode_SMD:D_SOD-123, symbol Device:D_Schottky_Small
- added H5: MOTA_Pad, MountingHole:MountingHole_4.3mm_M4_Pad, symbol Mechanical:MountingHole_Pad
- added H6: MOTB_Pad, MountingHole:MountingHole_4.3mm_M4_Pad, symbol Mechanical:MountingHole_Pad
- added H7: MOTC_Pad, MountingHole:MountingHole_4.3mm_M4_Pad, symbol Mechanical:MountingHole_Pad
- added L2: 68n, Inductor_SMD:L_0603_1608Metric, symbol Device:L_Small
- added Q1, Q2: AO3401A, Package_TO_SOT_SMD:SOT-23, symbol Transistor_FET:AO3401A
- C1: renamed from C?; footprint (none) -> Capacitor_SMD:C_0805_2012Metric; LCSC Part # (none) -> C28323; Vmax (none) -> 6.3
- C10: renamed from C?; footprint (none) -> Capacitor_SMD:C_0805_2012Metric; LCSC Part # (none) -> C28233; Vmax (none) -> 100
- C11, C12: renamed from C?; footprint (none) -> Capacitor_SMD:C_0805_2012Metric; LCSC Part # (none) -> C28323; Vmax (none) -> 16
- C13: renamed from C?; value 0.1u -> 100n; footprint (none) -> Capacitor_SMD:C_0402_1005Metric; LCSC Part # (none) -> C307331; Vmax (none) -> 6.3
- C14, C15: renamed from C?; footprint (none) -> Capacitor_SMD:C_0603_1608Metric; LCSC Part # (none) -> C23630; Vmax (none) -> 3.3
- C16: renamed from C?; footprint (none) -> Capacitor_SMD:C_0805_2012Metric; LCSC Part # (none) -> C472826; Vmax (none) -> 100
- C17, C18: renamed from C?; footprint (none) -> Capacitor_SMD:C_0402_1005Metric; LCSC Part # (none) -> C32949; Vmax (none) -> 3.3
- C19, C20: renamed from C?; footprint (none) -> Capacitor_SMD:C_0805_2012Metric; LCSC Part # (none) -> C28233; Vmax (none) -> 3.3
- C2: renamed from C?; footprint (none) -> Capacitor_SMD:C_0603_1608Metric; LCSC Part # (none) -> C19666; Vmax (none) -> 3.3
- C21: renamed from C?; footprint (none) -> Capacitor_SMD:C_0805_2012Metric; LCSC Part # (none) -> C472826; Vmax (none) -> 6.3
- C3, C4, C5, C6, C7, C9: renamed from C?; footprint (none) -> Capacitor_SMD:C_0402_1005Metric; LCSC Part # (none) -> C307331; Vmax (none) -> 3.3
- C8: renamed from C?; footprint (none) -> Capacitor_SMD:C_0805_2012Metric; LCSC Part # (none) -> C28323; Vmax (none) -> 3.3
- Cb1: renamed from Cb; footprint (none) -> Capacitor_SMD:C_0805_2012Metric; LCSC Part # (none) -> C1710; Vmax (none) -> 50
- Cbulk1, Cbulk2, Cbulk3: renamed from C?; Vmax (none) -> 100
- Cbyp1: renamed from Cbyp; footprint (none) -> Capacitor_SMD:C_0805_2012Metric; LCSC Part # (none) -> C28323; Vmax (none) -> 16
- Cbyp2, Cbyp3, Cbyp4: renamed from C?; value C_Small -> 0.1u; footprint (none) -> Capacitor_SMD:C_0805_2012Metric; LCSC Part # (none) -> C28233; Vmax (none) -> 100
- Cff1: renamed from Cff; footprint (none) -> Capacitor_SMD:C_0603_1608Metric; LCSC Part # (none) -> C458911; Vmax (none) -> 50
- Cin1: renamed from Cin; Vmax (none) -> 100
- Cinx1: renamed from Cinx; footprint (none) -> Capacitor_SMD:C_0805_2012Metric; LCSC Part # (none) -> C28233; Vmax (none) -> 100
- Cout1: renamed from Cout; footprint (none) -> Capacitor_SMD:C_0805_2012Metric; LCSC Part # (none) -> C15850; Vmax (none) -> 6.3
- D2, D3: renamed from D?; footprint (none) -> Diode_SMD:D_MiniMELF; LCSC Part # (none) -> C8062
- F1: renamed from F?; LCSC Part # (none) -> C12430
- FB1: renamed from FB?; footprint Capacitor_SMD:C_0805_2012Metric -> Inductor_SMD:L_0805_2012Metric; LCSC Part # (none) -> C1017
- H1, H2, H3, H4: renamed from H?; footprint (none) -> MountingHole:MountingHole_4.3mm_M4_Pad_Via
- IC1: renamed from IC?; footprint SOIC127P600X175-8N -> SamacSys_Parts:SOIC127P600X175-8N
- J1, J2, J5, J6: renamed from J?; footprint (none) -> Connector_Molex:Molex_PicoBlade_53047-0410_1x04_P1.25mm_Vertical
- J3: renamed from J?; footprint (none) -> Connector_PinSocket_1.27mm:PinSocket_2x05_P1.27mm_Vertical_SMD
- L1: footprint (none) -> Inductor_THT:L_Radial_D10.5mm_P5.00mm_Abacron_AISR-01; LCSC Part # (none) -> C122800
- LED1: renamed from D?; footprint (none) -> LED_SMD:LED_0603_1608Metric; LCSC Part # (none) -> C2286
- LED2: renamed from D?; footprint (none) -> LED_SMD:LED_0603_1608Metric; LCSC Part # (none) -> C2290
- R1: renamed from R?; value 4K7 -> 5k1; footprint (none) -> 0603; LCSC Part # (none) -> C23186
- R10, R11: renamed from R?; value 4k7 -> 5k1; footprint (none) -> 0603; LCSC Part # (none) -> C23186
- R15, R16: renamed from R?; footprint (none) -> 0603; LCSC Part # (none) -> C23186
- U3: renamed from U?; footprint QFN50P700X700X100-49N -> DRV8353RSRGZT:QFN50P700X700X100-49N
- gave numbers to parts that had none: 23
- renumbered RT to RT1, Rfbb to Rfbb1, Rfbt to Rfbt1, Rilim to Rilim1, Rseries to Rseries1
Connections:
- net +3.3VA: now also L2.2; no longer C19.2, C2.1, C20.1, C3.1, C4.1, C5.1, C6.1, C7.1, Cout1.1, IC1.3 (VDD), J1.1 (Pin_1), J2.1 (Pin_1), J3.1 (Pin_1), J5.1 (Pin_1), J6.1 (Pin_1), LED1.2 (A), R10.1, R11.1, R6.1, R7.2, Rseries1.2, SW1.1 (A), U1.1 (VBAT), U1.19 (VDD), U1.32 (VDD), U1.48 (VDD), U1.64 (VDD), U2.2 (VO), U3.26 (VREF)
- net +BATT: now also Q2.1 (G)
- net DRV:ENABLE: now also U1.17 (PA3)
- net DRV:INHA: now also U1.41 (PA8)
- net DRV:INHB: now also U1.42 (PA9)
- net DRV:INHC: now also U1.43 (PA10)
- net DRV:INLA: now also U1.34 (PB13)
- net DRV:INLB: now also U1.35 (PB14)
- net DRV:INLC: now also U1.36 (PB15)
- net DRV:nFAULT: now also U1.24 (PC4)
- net DRV:nSCS: now also U1.20 (PA4); no longer U1.24 (PC4)
- net GLA: now also Q4.1 (G)
- net GND: now also D1.2 (A)
- net LED_STATUS: now also U1.2 (PC13)
- net SOA: now also U1.9 (PC1)
- net SOB: now also U1.10 (PC2)
- net SOC: now also U1.11 (PC3)
- net SW: now also D1.1 (K)
- net USB_Vbus: now also Q2.3 (D)
- net at D2.2 (A), R2.1: now also Q1.1 (G)
- net at D3.1 (K), U2.3 (VI): now also Q2.2 (S)
- net at D2.1 (K), FB1.1: now also Q1.2 (S)
- net at F1.1: now also Q1.3 (D)
- net MOTA renamed SHA
- net SHA: now also H5.1
- net MOTB renamed SHB
- net SHB: now also H6.1
- net MOTC renamed SHC
- net SHC: now also H7.1
- new net +3V3: C19.2, C2.1, C20.1, C3.1, C4.1, C5.1, C6.1, C7.1, Cout1.1, IC1.3 (VDD), J1.1 (Pin_1), J2.1 (Pin_1), J3.1 (Pin_1), J5.1 (Pin_1), J6.1 (Pin_1), L2.1, LED1.2 (A), R10.1, R11.1, R6.1, R7.2, Rseries1.2, SW1.1 (A), U1.1 (VBAT), U1.19 (VDD), U1.32 (VDD), U1.48 (VDD), U1.64 (VDD), U2.2 (VO), U3.26 (VREF)
- no-connect marks 4 -> 23
Other:
- note added: "Basic LPF: 68nH and 1.1uC gives a corner F of: 582kHz"
- note added: "From USB"
- note added: "If+BATT voltage is present, then: PMOS reverse biased and turns off ∴ draw from USB 5V disabled so no PSU backfeeding occurs (that could damage USB)"
- note added: "MCU power supply: From battery"
- note added: "Switches, Moter Output & Feedback"
- note removed: "If+BATT voltage is present, then: PMOS reverse biased and turns off ∴ draw from USB 5V disabled so no PSU backfeeding occurs (and damages USB)"
- note removed: "MCU power supply:"
- note removed: "Switches & Feedback"
- moved on the sheet: C18, C2, C3, C4, C5, C6, C7, C8, C9, Cbulk1, Cbulk3, Cbyp2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

Commit message: Finished BOM
Parts:
- added R14, R18: 120, Resistor_SMD:R_0603_1608Metric, symbol Device:R_Small
- C1, C10, C11, C12, C13, C14, C15, C17, C18, C19, C2, C20, C3, C4, C5, C6, C7, C8, C9, Cb1, Cbyp1, Cbyp2, Cbyp3, Cbyp4, Cinx1, Cout1, FB1, L2, LED1, LED2, Q1, Q2: Basic/Extended (none) -> Bas
- C16, C21, Cff1, D1, F1, L1: Basic/Extended (none) -> Ext
- D2, D3: value D_Z -> 5V6; Basic/Extended (none) -> Bas
- J1, J2, J5, J6: Basic/Extended (none) -> Ext; LCSC Part # (none) -> C504989
- J3: Basic/Extended (none) -> Ext; LCSC Part # (none) -> C2684733
- J4: Basic/Extended (none) -> Ext; LCSC Part # (none) -> C165948
- Q3, Q4, Q5, Q6, Q7, Q8: footprint (none) -> Package_TO_SOT_THT:TO-220-3_Horizontal_TabDown; Mouser Part Number (none) -> 942-IRFB4110PBF; Mouser Price/Stock (none) -> https://www.mouser.com/ProductDetail/Infineon-IR/IRFB4110PB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
- R1, R10, R11: footprint 0603 -> Resistor_SMD:R_0603_1608Metric; Basic/Extended (none) -> Bas
- R12: footprint (none) -> Resistor_SMD:R_0603_1608Metric; Basic/Extended (none) -> Bas; LCSC Part # (none) -> C21190
- R13, R4, R9: value 0.01 -> 0.001; footprint (none) -> DRV8353RSRGZT:R_3920_1127Metric
- R15: renamed from R14; value 60 -> 120; footprint (none) -> Resistor_SMD:R_0603_1608Metric; Basic/Extended (none) -> Bas; LCSC Part # (none) -> C22787
- R16: renamed from R15; footprint 0603 -> Resistor_SMD:R_0603_1608Metric; Basic/Extended (none) -> Bas
- R17: renamed from R16; footprint 0603 -> Resistor_SMD:R_0603_1608Metric; Basic/Extended (none) -> Bas
- R19: renamed from R17; value 60 -> 120; footprint (none) -> Resistor_SMD:R_0603_1608Metric; Basic/Extended (none) -> Bas; LCSC Part # (none) -> C22787
- R2, R3: value 100k -> 133k; footprint (none) -> Resistor_SMD:R_0603_1608Metric; Basic/Extended (none) -> Ext; LCSC Part # (none) -> C22870
- R5, R6, Rfbt1: footprint (none) -> Resistor_SMD:R_0603_1608Metric; Basic/Extended (none) -> Bas; LCSC Part # (none) -> C25804
- R7: value 1k -> 5k1; footprint (none) -> Resistor_SMD:R_0603_1608Metric; Basic/Extended (none) -> Bas; LCSC Part # (none) -> C23186
- R8: footprint (none) -> Resistor_SMD:R_0402_1005Metric; Basic/Extended (none) -> Bas; LCSC Part # (none) -> C25118
- RT1: footprint (none) -> Resistor_SMD:R_0603_1608Metric; Basic/Extended (none) -> Ext; LCSC Part # (none) -> C22949
- Rfbb1: footprint (none) -> Resistor_SMD:R_0603_1608Metric; Basic/Extended (none) -> Ext; LCSC Part # (none) -> C25967
- Rilim1: footprint (none) -> Resistor_SMD:R_0603_1608Metric; Basic/Extended (none) -> Ext; LCSC Part # (none) -> C22870
- Rseries1: footprint (none) -> Resistor_SMD:R_0805_2012Metric; Basic/Extended (none) -> Ext; LCSC Part # (none) -> C17373
- SW1: footprint (none) -> Button_Switch_SMD:SW_SPDT_PCM12; Basic/Extended (none) -> Ext; LCSC Part # (none) -> C221841
- U1: Basic/Extended (none) -> Ext; LCSC Part # (none) -> C15742
- U2: Basic/Extended (none) -> Bas; LCSC Part # (none) -> C6186
- U3: Basic/Extended (none) -> Ext; LCSC Part # (none) -> C2150650; Mouser Part Number (none) -> 595-DRV8353RSRGZT; Mouser Price/Stock (none) -> https://www.mouser.com/ProductDetail/Texas-Instruments/DRV8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
- U4: Basic/Extended (none) -> Ext; LCSC Part # (none) -> C7519
- Y1: footprint (none) -> Crystal:Crystal_SMD_3225-4Pin_3.2x2.5mm; Basic/Extended (none) -> Bas; LCSC Part # (none) -> C13738
Connections:
- net at C21.1, R15.2, R19.1: now also R14.2, R18.1
- net at IC1.6 (CANL), J2.3 (Pin_3), R19.2: now also R18.2
- net at IC1.7 (CANH), J2.2 (Pin_2), R15.1: now also R14.1
Other:
- note added: "MCU Connectors"
- note added: "Power LED: 2V drop over LED 3.3V - 2V = 1.3V 5.1kOhm -> 1.3/5.1k = 0.255mA"
- note removed: "Connectors"
- note removed: "Power LED: 2V drop over LED 3.3V - 2V = 1.3V 4.7kOhm -> 1.3/4.7k = 0.277mA"
- moved on the sheet: C20, C21, IC1, R15, R19
